File: Hardware/Schematic/JTAG.sch (KiCad schematic (older format))
At the start: 7 parts, among them J3 JTAG, J4 Conn_02x04_Odd_Even, J5 Conn_02x02_Odd_Even

Commit message: Lots of schematic updates
Lots of stuff...

* Added a new 8-pin TVS diode array
* Finalized the display connector
* Corrected the net labels to global labels so they span across sheets
* Added a 5V linear voltage regulator and LEDs to debug power
Connections:
- no-connect marks 0 -> 3
Changed lines of the file:
@@
 $Descr A4 11693 8268
 encoding utf-8
-Sheet 2 5
+Sheet 2 6
 Title ""
 Date ""
@@
 Wire Wire Line
 	3450 4250 3450 4300
-Text Label 6300 3450 0    50   ~ 0
-JTAG_TRST|SPI1_MISO|TIM3_CH1
-Text Label 6300 3650 0    50   ~ 0
-JTAG_TMS
-Text Label 6300 3750 0    50   ~ 0
-JTAG_TCK
-Text Label 6300 4050 0    50   ~ 0
-RST
 Wire Wire Line
 	4150 3850 4350 3850
 Wire Wire Line
 	4350 3850 4350 4250
-Text Label 6300 3950 0    50   ~ 0
-JTAG_TDO|SPI1_SCK|I2S3_SCK
-Text Label 6300 3550 0    50   ~ 0
-JTAG_TDI|SPI1_SS|I2S3_WS
 Wire Wire Line
 	4400 3450 5500 3450
@@
 	1    0    0    -1
 $EndComp
+NoConn ~ 3650 3350
+NoConn ~ 4150 4150
+NoConn ~ 4150 4250
+Text GLabel 6300 3450 2    50   BiDi ~ 0
+JTAG_TRST|SPI1_MISO|TIM3_CH1
+Text GLabel 6300 3550 2    50   BiDi ~ 0
+JTAG_TDI|SPI1_SS|I2S3_WS
+Text GLabel 6300 3650 2    50   BiDi ~ 0
+JTAG_TMS
+Text GLabel 6300 3750 2    50   BiDi ~ 0
+JTAG_TCK
+Text GLabel 6300 3950 2    50   BiDi ~ 0
+JTAG_TDO|SPI1_SCK|I2S3_SCK
+Text GLabel 6300 4050 2    50   BiDi ~ 0
+RST
 $EndSCHEMATC
