File: Hardware/Schematic/Photon/Particle_Connector.sch (KiCad schematic (older format))
At the start: 18 parts, among them J1 Conn_01x12, J11 Conn_01x01, J12 Conn_01x01, J13 Conn_01x32, J14 Conn_01x01, J15 Conn_01x01, J16 Conn_01x01, J17 Conn_01x01, J18 Conn_01x01, J2 Conn_01x12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

Commit message: Split-up schematics into three seperate projects with a parts library as well
Parts:
- D1, D2, D3, D4: symbol WiFiLMR-rescue:ESDA6V1U1-Power_Protection -> parts:ESDA6V1U1-Power_Protection
Changed lines of the file:
@@
 $Descr A4 11693 8268
 encoding utf-8
-Sheet 3 6
+Sheet 3 5
 Title ""
 Date ""
@@
 	6050 5200 6050 5000
 $Comp
-L WiFiLMR-rescue:ESDA6V1U1-Power_Protection D4
+L parts:ESDA6V1U1-Power_Protection D4
 U 1 1 5CFE731E
 P 10400 4750
@@
 $EndComp
 $Comp
-L WiFiLMR-rescue:ESDA6V1U1-Power_Protection D3
+L parts:ESDA6V1U1-Power_Protection D3
 U 1 1 5CFF73FC
 P 9700 4750
@@
 $EndComp
 $Comp
-L WiFiLMR-rescue:ESDA6V1U1-Power_Protection D2
+L parts:ESDA6V1U1-Power_Protection D2
 U 1 1 5D000224
 P 1950 4700
@@
 $EndComp
 $Comp
-L WiFiLMR-rescue:ESDA6V1U1-Power_Protection D1
+L parts:ESDA6V1U1-Power_Protection D1
 U 1 1 5D00022A
 P 1250 4700

Commit message: Updated keypad and display schematic to use header sockets for intra-board connections.
Parts:
- J13: footprint Connector_PinHeader_1.00mm:PinHeader_1x32_P1.00mm_Horizontal -> Connector_PinHeader_2.54mm:PinHeader_2x16_P2.54mm_Horizontal
Changed lines of the file:
@@
 F 0 "J13" V 4075 7046 50  0000 C CNN
 F 1 "Conn_01x32" V 4166 7046 50  0000 C CNN
-F 2 "Connector_PinHeader_1.00mm:PinHeader_1x32_P1.00mm_Horizontal" H 3950 7100 50  0001 C CNN
+F 2 "Connector_PinHeader_2.54mm:PinHeader_2x16_P2.54mm_Horizontal" H 3950 7100 50  0001 C CNN
 F 3 "~" H 3950 7100 50  0001 C CNN
 	1    3950 7100
